File: Proyecto/Proyecto.kicad_pcb (KiCad board)
At the start: 2 copper layers, 104.1 x 96.5 mm, 48 parts, among them IC1 MC9S08MP16xLC, J1 Bomba1, J10 DHT11, J11 Bomba2, J12 Aux1, J13 LCD, J14 Aux2, J15 Expansion, J16 NIVEL BAJO, J17 NIVEL ALTO, J18 LDR, J2 Rele1, J3 Luces, J4 Rele2, J5 TDS, J6 Rele3, J7 Rele4, J8 ENTRADA, J9 PH, K1 FINDER-36.11, K2 FINDER-36.11, K3 FINDER-36.11, K4 FINDER-36.11, Q1 IRF3205, Q2 IRF3205, U1 ULN2803A, U2 MIC4427, U3 AP63205WU, U4 PC817, U5 PC817, U6 LM358, U7 LM358

Commit message: 7-8-2022 itLA
Parts:
- moved J6 140.5 mm to (71.1, 141.0), turned to 0 degrees
- moved J4 139.5 mm to (54.6, 141.0), turned to 0 degrees
- moved J2 138.5 mm to (38.1, 141.0), turned to 0 degrees
- moved J5 126.1 mm to (48.3, 78.7), turned to 180 degrees
- moved J7 122.9 mm to (87.6, 141.0), turned to 0 degrees
- moved J9 97.0 mm to (64.8, 78.7), turned to 180 degrees
- moved U1 96.1 mm to (54.6, 104.1)
- moved U6 92.9 mm to (72.4, 105.4)
- moved U7 92.9 mm to (82.5, 105.4)
- moved K1 92.8 mm to (43.2, 118.5), turned to -90 degrees
- moved J11 90.4 mm to (104.1, 141.0), turned to 0 degrees
- moved J1 84.6 mm to (115.6, 141.0), turned to 0 degrees
- moved J18 75.6 mm to (115.6, 78.7), turned to 180 degrees
- moved RV1 73.1 mm to (102.9, 109.2)
- moved K2 68.7 mm to (59.7, 118.5), turned to -90 degrees
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Connections:
- J2 pad 1: Net-(J2-Pad1) -> Net-(K1-Pad14)
- J2 pad 2: Net-(J2-Pad2) -> Net-(K1-Pad11)
- J2 pad 3: Net-(J2-Pad3) -> Net-(K1-Pad12)
- J4 pad 2: Net-(J4-Pad2) -> Net-(K2-Pad11)
- J4 pad 3: Net-(J4-Pad3) -> Net-(K2-Pad12)
- J6 pad 1: Net-(J6-Pad1) -> Net-(K3-Pad14)
- J6 pad 2: Net-(J6-Pad2) -> Net-(K3-Pad11)
- J6 pad 3: Net-(J6-Pad3) -> Net-(K3-Pad12)
- J7 pad 1: Net-(J7-Pad1) -> Net-(K4-Pad14)
- J7 pad 2: Net-(J7-Pad2) -> Net-(K4-Pad11)
- J7 pad 3: Net-(J7-Pad3) -> Net-(K4-Pad12)
- K1 pad 11: Net-(J2-Pad3) -> Net-(K1-Pad11)
- K1 pad 12: Net-(J2-Pad1) -> Net-(K1-Pad12)
- K1 pad 14: Net-(J2-Pad2) -> Net-(K1-Pad14)
- K2 pad 11: Net-(J4-Pad3) -> Net-(K2-Pad11)
- K2 pad 12: Net-(J4-Pad1) -> Net-(K2-Pad12)
- K2 pad 14: Net-(J4-Pad2) -> Net-(J4-Pad1)
- K3 pad 11: Net-(J6-Pad3) -> Net-(K3-Pad11)
- K3 pad 12: Net-(J6-Pad1) -> Net-(K3-Pad12)
- K3 pad 14: Net-(J6-Pad2) -> Net-(K3-Pad14)
- K4 pad 11: Net-(J7-Pad3) -> Net-(K4-Pad11)
- K4 pad 12: Net-(J7-Pad1) -> Net-(K4-Pad12)
- K4 pad 14: Net-(J7-Pad2) -> Net-(K4-Pad14)
- R3 pad 1: unconnected-(R3-Pad1) -> +5V
- R4 pad 1: unconnected-(R4-Pad1) -> +5V
Routing:
- net Net-(J3-Pad2): track 0.00 -> 16.1 mm
- net Net-(J3-Pad1): track 0.00 -> 14.5 mm
- net GND: track 0.00 -> 12.5 mm
Other:
- board outline removed

Commit message: 15-7-2022
Parts:
- added C10: 100n, Capacitor_SMD:C_0201_0603Metric, F.Cu at (89.5, 130.2)
- added C11: 100n, Capacitor_SMD:C_0201_0603Metric, F.Cu at (106.7, 127.0)
- added C8: 30p, Capacitor_SMD:C_0201_0603Metric, F.Cu at (106.0, 121.9)
- added C9: 30p, Capacitor_SMD:C_0201_0603Metric, F.Cu at (93.3, 134.0)
- added HOLE3: MountingHole_2.2mm_M2, MountingHole:MountingHole_2.2mm_M2, F.Cu at (181.0, 165.1)
- added HOLE3: MountingHole_2.2mm_M2, MountingHole:MountingHole_2.2mm_M2, F.Cu at (37.5, 165.1)
- added HOLE3: MountingHole_2.2mm_M2, MountingHole:MountingHole_2.2mm_M2, F.Cu at (181.0, 99.7)
- added HOLE3: MountingHole_2.2mm_M2, MountingHole:MountingHole_2.2mm_M2, F.Cu at (37.5, 99.7)
- added L2: 27n, Inductor_SMD:L_0805_2012Metric, F.Cu at (112.6, 14.1)
- added R10: 10K, Resistor_SMD:R_0201_0603Metric, F.Cu at (67.4, 63.2)
- added R11: 10K, Resistor_SMD:R_0201_0603Metric, F.Cu at (106.8, 20.3)
- added R8: 1M, Resistor_SMD:R_0201_0603Metric, F.Cu at (83.4, 46.3)
- added R9: 10K, Resistor_SMD:R_0201_0603Metric, F.Cu at (93.3, 35.8)
- added RV2: Varistor_6V, Capacitor_SMD:C_0805_2012Metric, F.Cu at (84.4, 41.4)
- added U8: ULN2003A, Package_SO:SOIC-16_3.9x9.9mm_P1.27mm, F.Cu at (135.3, 143.5)
- added Y1: Crystal 4 MHz, Crystal:Crystal_HC49-4H_Vertical, F.Cu at (54.8, 34.2)
- C1, C4, C5: footprint Capacitor_SMD:C_0603_1608Metric -> Capacitor_SMD:C_0805_2012Metric
- C3: footprint Capacitor_SMD:C_0603_1608Metric -> Capacitor_SMD:C_0201_0603Metric
- J1: value Bomba1 -> Conn_01x12_Male; footprint TerminalBlock:TerminalBlock_bornier-2_P5.08mm -> Connector_PinHeader_2.54mm:PinHeader_1x12_P2.54mm_Vertical
- J11: value Bomba2 -> Bomba1
- J12: value Aux1 -> Bomba2
- J14: value Aux2 -> Aux1
- J15: value Expansion -> Aux2; footprint Connector_PinHeader_1.00mm:PinHeader_1x10_P1.00mm_Vertical -> TerminalBlock:TerminalBlock_bornier-2_P5.08mm
- L1: value L -> 4.7u; footprint Inductor_SMD:L_0603_1608Metric -> Inductor_SMD:L_Bourns_SRN6045TA
- U1: value ULN2803A -> ULN2003A; footprint Package_SO:SOIC-18W_7.5x11.6mm_P1.27mm -> Package_SO:SOIC-16_3.9x9.9mm_P1.27mm
- moved R1 97.5 mm to (57.1, 67.0)
- moved R2 90.9 mm to (61.1, 66.1)
- moved RV1 85.6 mm to (102.5, 23.6)
- moved J15 84.9 mm to (138.4, 163.2), turned to 0 degrees
- moved R7 78.0 mm to (75.8, 54.0), turned to 0 degrees
- moved J1 68.2 mm to (177.8, 113.0)
- moved J5 66.3 mm to (110.5, 101.6)
- moved J13 56.6 mm to (171.4, 124.2), turned to 0 degrees
- moved U7 52.7 mm to (96.5, 54.6)
- moved J4 49.1 mm to (98.4, 163.2)
- moved C2 48.9 mm to (87.0, 119.4)
- moved K2 48.8 mm to (103.5, 139.9)
- moved R3 47.6 mm to (60.2, 63.5)
- moved R5 45.5 mm to (84.2, 44.2)
- moved C6 42.9 mm to (88.3, 125.1)
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Connections:
- IC1 pad 12: unconnected-(IC1-Pad12) -> BKGD_PIN
- IC1 pad 21: unconnected-(IC1-Pad21) -> Net-(IC1-Pad21)
- IC1 pad 22: unconnected-(IC1-Pad22) -> GND
- IC1 pad 27: unconnected-(IC1-Pad27) -> Net-(IC1-Pad27)
- IC1 pad 28: unconnected-(IC1-Pad28) -> Net-(IC1-Pad28)
- IC1 pad 29: unconnected-(IC1-Pad29) -> GND
- IC1 pad 30: unconnected-(IC1-Pad30) -> Reset_pin
- IC1 pad 6: unconnected-(IC1-Pad6) -> GND
- IC1 pad 7: unconnected-(IC1-Pad7) -> +5V
- J1 pad 1: Net-(J1-Pad1) -> RX
- J1 pad 2: +12V -> TX
- J15 pad 1: RX -> Net-(J15-Pad1)
- J15 pad 2: TX -> +12V
- K1 pad A1: GND -> +12V
- K2 pad A1: GND -> +12V
- K3 pad A1: GND -> +12V
- K4 pad A1: GND -> +12V
- U1 pad 10: +12V -> unconnected-(U1-Pad10)
- U1 pad 11: Net-(J14-Pad1) -> unconnected-(U1-Pad11)
- U1 pad 12: Net-(J12-Pad1) -> unconnected-(U1-Pad12)
- U1 pad 13: Net-(J11-Pad1) -> Net-(K4-PadA2)
- U1 pad 14: Net-(J1-Pad1) -> Net-(K3-PadA2)
- U1 pad 15: Net-(K4-PadA2) -> Net-(K2-PadA2)
- U1 pad 16: Net-(K3-PadA2) -> Net-(K1-PadA2)
- U1 pad 5: Bomba1 -> unconnected-(U1-Pad5)
- U1 pad 6: Bomba2 -> unconnected-(U1-Pad6)
- U1 pad 7: Aux1 -> unconnected-(U1-Pad7)
- U1 pad 8: Aux2 -> GND
- U1 pad 9: GND -> +12V
Routing:
- net Net-(J3-Pad2): track 16.1 -> 0.00 mm
- net Net-(J3-Pad1): track 14.5 -> 0.00 mm
- net GND: track 12.5 -> 0.00 mm
Other:
- board text removed: "JOSE PCB"

Commit message: 7-15-2022 ITLA
Parts:
- removed R9: 10K, Resistor_SMD:R_0201_0603Metric
- J1: value Conn_01x12_Male -> Conn_01x09_Male; footprint Connector_PinHeader_2.54mm:PinHeader_1x12_P2.54mm_Vertical -> Connector_PinSocket_2.54mm:PinSocket_1x09_P2.54mm_Vertical
- J13: footprint Connector_PinHeader_1.00mm:PinHeader_1x04_P1.00mm_Vertical -> Connector_PinHeader_2.54mm:PinHeader_1x04_P2.54mm_Vertical
- moved L2 114.3 mm to (134.6, 126.3), turned to 90 degrees
- moved R11 105.0 mm to (128.3, 123.1)
- moved Y1 104.9 mm to (119.5, 116.8)
- moved R5 98.8 mm to (141.8, 124.4)
- moved RV1 82.5 mm to (129.5, 101.6)
- moved RV2 75.1 mm to (114.0, 110.4)
- moved R8 74.8 mm to (121.9, 110.4)
- moved R10 71.2 mm to (101.6, 125.7)
- moved U7 71.2 mm to (55.9, 113.0)
- moved R7 69.7 mm to (48.3, 118.1)
- moved R1 68.9 mm to (108.4, 113.0)
- moved U6 67.2 mm to (101.6, 113.0)
- moved R4 66.2 mm to (91.4, 126.1)
- moved R3 61.1 mm to (94.4, 114.2)
- moved U2 57.8 mm to (105.4, 130.7)
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Connections:
- net Net-(C3-Pad1) renamed /SW
- IC1 pad 27: Net-(IC1-Pad27) -> Net-(C8-Pad2)
- J1 pad 6: ADC -> +5V
- J1 pad 7: Digital -> Reset_pin
- J1 pad 8: Digital_1 -> BKGD_PIN
- J1 pad 9: +5V -> GND
Routing:
- net Net-(J7-Pad2): track 0.00 -> 23.3 mm
- net Net-(J6-Pad2): track 0.00 -> 23.3 mm
- net Net-(J4-Pad2): track 0.00 -> 23.3 mm
- net Net-(J2-Pad2): track 0.00 -> 23.3 mm
- net Net-(C8-Pad2): track 0.00 -> 18.5 mm
- net Net-(C9-Pad2): track 0.00 -> 17.7 mm
- net +12V: track 0.00 -> 11.7 mm, vias 0 -> 8
- net Net-(J7-Pad1): track 0.00 -> 9.47 mm
- net Net-(J4-Pad3): track 0.00 -> 9.47 mm
- net Net-(J4-Pad1): track 0.00 -> 9.47 mm
- net Net-(J2-Pad3): track 0.00 -> 9.47 mm
- net Net-(J6-Pad1): track 0.00 -> 9.47 mm
- net Net-(J2-Pad1): track 0.00 -> 9.47 mm
- net Net-(J7-Pad3): track 0.00 -> 9.47 mm
- net Net-(J6-Pad3): track 0.00 -> 9.47 mm
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- added copper zone on F.Cu, net +12V
- added copper zone on In2.Cu, net +12V
- added copper zone on F.Cu, net +5V
- added copper zone on In2.Cu, net +5V
- added copper zone on F.Cu, net /SW
- added copper zone on F.Cu, net GND
- added copper zone on In1.Cu, net GND
Other:
- copper layers 2 -> 4

Commit message: 22-7-2022
Parts:
- moved J1 162.1 mm to (37.6, 131.0), turned to 90 degrees
- moved J13 155.4 mm to (37.6, 127.3), turned to 90 degrees
- moved RV1 55.9 mm to (74.7, 112.2)
- moved R6 52.2 mm to (118.5, 106.5), turned to 0 degrees
- moved C7 45.1 mm to (82.3, 122.7), turned to -90 degrees
- moved R11 44.6 mm to (84.0, 117.3), turned to 180 degrees
- moved U5 43.5 mm to (115.2, 107.3), turned to -90 degrees
- moved U4 41.3 mm to (124.7, 108.5), turned to -90 degrees
- moved J5 39.3 mm to (82.6, 101.6)
- moved R1 38.8 mm to (69.7, 110.3), turned to -90 degrees
- moved L2 38.4 mm to (96.3, 123.8), turned to 180 degrees
- moved C11 36.3 mm to (95.1, 122.0), turned to -90 degrees
- moved U6 35.9 mm to (65.7, 112.0), turned to -90 degrees
- moved U2 35.6 mm to (141.0, 130.0)
- moved J11 34.2 mm to (149.8, 163.3)
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Connections:
- IC1 pad 1: Nivel_bajo -> TDS
- IC1 pad 13: Rele1 -> Rele4
- IC1 pad 14: Rele2 -> Rele3
- IC1 pad 15: Rele3 -> Rele2
- IC1 pad 16: Rele4 -> Rele1
- IC1 pad 17: PH -> Nivel_alto
- IC1 pad 18: TDS -> Nivel_bajo
- IC1 pad 19: ldr -> Digital
- IC1 pad 2: Nivel_alto -> PH
- IC1 pad 3: Digital -> ldr
- IC1 pad 31: LUZ_B -> luz b
- IC1 pad 32: LUZ_A -> luz a
- IC1 pad 4: DHT11 -> DHt11
- J1 pad 1: RX -> +5V
- J1 pad 2: TX -> GND
- J1 pad 5: GND -> RX
- J1 pad 6: +5V -> TX
- J10 pad 1: Dht11 -> GND
- J10 pad 3: GND -> DHt11
- U1 pad 13: Net-(K4-PadA2) -> Net-(K1-PadA2)
- U1 pad 14: Net-(K3-PadA2) -> Net-(K4-PadA2)
- U1 pad 15: Net-(K2-PadA2) -> Net-(K3-PadA2)
- U1 pad 16: Net-(K1-PadA2) -> Net-(K2-PadA2)
- U2 pad 2: Luz_A -> luz a
- U2 pad 4: Luz_B -> luz b
Routing:
- net GND: track 1.32 -> 90.3 mm, vias 16 -> 29
- net luz a: track 0.00 -> 88.7 mm, vias 0 -> 4
- net Bomba1: track 0.00 -> 73.5 mm, vias 0 -> 2
- net luz b: track 0.00 -> 68.7 mm, vias 0 -> 4
- net SDA: track 0.00 -> 68.1 mm, vias 0 -> 3
- net Bomba2: track 0.00 -> 64.9 mm, vias 0 -> 2
- net Aux1: track 0.00 -> 60.5 mm, vias 0 -> 2
- net Rele4: track 0.00 -> 59.5 mm, vias 0 -> 6
- net Aux2: track 0.00 -> 58.8 mm, vias 0 -> 2
- net SCL: track 0.00 -> 52.7 mm, vias 0 -> 1
- net Reset_pin: track 0.00 -> 51.0 mm, vias 0 -> 5
- net Nivel_bajo: track 0.00 -> 49.5 mm, vias 0 -> 2
- net PH: track 0.00 -> 46.4 mm, vias 0 -> 2
- net Net-(K2-PadA2): track 0.00 -> 45.9 mm, vias 0 -> 2
- net DHt11: track 0.00 -> 44.6 mm, vias 0 -> 5
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
Commit message: gg
Parts:
- removed RV1: R_Potentiometer, Potentiometer_SMD:Potentiometer_Bourns_3314G_Vertical
- added C12: 4.7µ, Capacitor_SMD:C_0805_2012Metric, F.Cu at (194.8, 85.6)
- added C13: 100n, Capacitor_SMD:C_0201_0603Metric, F.Cu at (194.7, 84.0)
- added C14: 100n, Capacitor_SMD:C_0201_0603Metric, F.Cu at (136.1, 74.7)
- added C15: 100n, Capacitor_SMD:C_0201_0603Metric, F.Cu at (133.6, 78.3)
- added R12: 10K, Resistor_SMD:R_0201_0603Metric, F.Cu at (166.7, 81.2)
- added R13: 10K, Resistor_SMD:R_0201_0603Metric, F.Cu at (166.7, 82.3)
- added R14: 10, Resistor_SMD:R_0201_0603Metric, F.Cu at (208.0, 87.5)
- added R15: 10, Resistor_SMD:R_0201_0603Metric, F.Cu at (208.1, 86.3)
- added R16: 10, Resistor_SMD:R_0201_0603Metric, F.Cu at (202.7, 94.3)
- added R17: 10, Resistor_SMD:R_0201_0603Metric, F.Cu at (202.6, 95.7)
- added R18: 10K, Resistor_SMD:R_0201_0603Metric, F.Cu at (209.7, 87.5)
- added R19: 10K, Resistor_SMD:R_0201_0603Metric, F.Cu at (204.5, 95.7)
- added R20: 100K, Resistor_SMD:R_0201_0603Metric, F.Cu at (97.9, 56.8)
- added R9: 10K, Resistor_SMD:R_0201_0603Metric, F.Cu at (166.8, 79.6)
- added SW1: SW_DIP_x04, Button_Switch_SMD:SW_DIP_SPSTx04_Slide_9.78x12.34mm_W8.61mm_P2.54mm, F.Cu at (159.1, 92.8)
- J1: footprint Connector_PinSocket_2.54mm:PinSocket_1x09_P2.54mm_Vertical -> Connector_PinHeader_2.54mm:PinHeader_1x09_P2.54mm_Vertical
- moved U2 67.1 mm to (194.8, 89.9)
- moved C10 67.0 mm to (138.0, 69.3)
- moved C11 67.0 mm to (136.6, 69.4)
- moved RV2 67.0 mm to (141.1, 69.3)
- moved L2 67.0 mm to (137.8, 71.1)
- moved J11 66.6 mm to (190.3, 110.4)
- moved J7 66.5 mm to (103.4, 110.4)
- moved J15 66.5 mm to (156.2, 110.4)
- moved J4 66.5 mm to (138.9, 110.4)
- moved J3 66.5 mm to (201.8, 110.5)
- moved J2 66.5 mm to (85.6, 110.5)
- moved J6 66.5 mm to (121.1, 110.5)
- moved J12 66.4 mm to (178.9, 110.5)
- moved J14 66.3 mm to (167.5, 110.5)
- moved C2 65.6 mm to (123.0, 67.2)
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Connections:
- U2 pad 5: Net-(Q2-Pad1) -> Net-(U2-Pad5)
- U2 pad 6: +5V -> +12V
- U2 pad 7: Net-(Q1-Pad1) -> Net-(U2-Pad7)
Routing:
- net Digital_1: track 0.00 -> 59.1 mm, vias 0 -> 5
- net +5V: track 39.8 -> 94.3 mm, vias 36 -> 27
- net ADC: track 0.00 -> 49.3 mm
- net Digital: track 0.00 -> 44.8 mm, vias 0 -> 4
- net Net-(Q1-Pad1): track 40.6 -> 5.34 mm, vias 3 -> 0
- net GND: track 90.3 -> 122.0 mm, vias 29 -> 33
- net Net-(Q2-Pad1): track 35.1 -> 4.90 mm, vias 1 -> 0
- net luz a: track 88.7 -> 106.6 mm
- net luz b: track 68.7 -> 86.7 mm
- net Net-(U2-Pad5): track 0.00 -> 15.9 mm, vias 0 -> 2
- net Net-(U2-Pad7): track 0.00 -> 11.3 mm
- net +12V: track 14.0 -> 21.5 mm, vias 9 -> 11
- net Net-(J18-Pad1): track 33.9 -> 27.1 mm, vias 4 -> 2
- net Net-(J17-Pad1): track 6.50 -> 10.8 mm, vias 0 -> 2
- net Net-(J15-Pad1): track 24.2 -> 26.9 mm
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Other:
- board text added: "+12V"
- board text added: "+5V"
- board text added: "BOMBA1"
- board text added: "BOMBA2"
- board text added: "COM"
- board text added: "DHT11"
- board text added: "EXPANSION"
- board text added: "GND"
- board text added: "LCD"
- board text added: "LDR"
- board text added: "LUZ_A"
- board text added: "LUZ_B"
- board text added: "M1"
- board text added: "M2"
- board text added: "NC"
- board text added: "NIVEL A"
- board text added: "NIVEL B"
- board text added: "NO"
- board text added: "PH"
- board text added: "TDS"
