File: Proyecto/Proyecto.kicad_sch (KiCad schematic)
At the start: 19 parts

Commit message: 30-6-2022
Parts:
- removed J? (x2): Conn_01x03, symbol Connector_Generic:Conn_01x03
- removed J?: Conn_01x04, symbol Connector_Generic:Conn_01x04
- removed J?: Conn_01x02, symbol Connector_Generic:Conn_01x02
- added C?: 100nF, symbol Device:C
- added IC?: MC9S08MP16xLC, Package_QFP:LQFP-32_7x7mm_P0.8mm, symbol MCU_NXP_S08:MC9S08MP16xLC
- added J?: Conn_01x04_Male, symbol Connector:Conn_01x04_Male
- added J? (x5): Conn_01x03, symbol Connector_Generic:Conn_01x03
- added J?: Conn_01x08, symbol Connector_Generic:Conn_01x08
- added K? (x4): FINDER-36.11, Relay_THT:Relay_SPDT_Finder_36.11, symbol Relay:FINDER-36.11
- added R?: 1k, symbol Device:R
- added SW?: SW_DIP_x03, symbol Switch:SW_DIP_x03
- added U?: MIC4427, symbol Driver_FET:MIC4427
Connections:
- net +12V: now also J?.1 (Pin_1)
- net +5V: now also J?.2 (Pin_2), J?.2 (Pin_2), J?.2 (Pin_2), U?.10 (COM), K?.A1, K?.A1, K?.A1, K?.A1, U?.6 (V+)
- net GND: now also J?.1 (Pin_1), J?.1 (Pin_1), J?.2 (Pin_2), J?.3 (Pin_3), Q?.3 (S), Q?.3 (S), C?.2, J?.3 (Pin_3), J?.5 (Pin_5), J?.6 (Pin_6), J?.7 (Pin_7), J?.8 (Pin_8), U?.3 (GND)
- net Rele1: now reaches U?.1 (I1)
- net Rele1: now also IC?.13 (PTA4)
- net at U?.11 (O8): now also J?.4 (Pin_4)
- net at U?.12 (O7): now also J?.3 (Pin_3)
- net at U?.13 (O6): now also J?.2 (Pin_2)
- net at U?.14 (O5): now also J?.1 (Pin_1)
- net at U?.15 (O4): now also K?.A2
- net at U?.16 (O3): now also K?.A2
- net at U?.17 (O2): now also K?.A2
- net at U?.18 (O1): now also K?.A2
- net Rele2: now reaches U?.2 (I2)
- net Rele2: now also IC?.14 (PTA5)
- net Rele3: now reaches U?.3 (I3)
- net Rele3: now also IC?.15 (PTA6)
- net Rele4: now reaches U?.4 (I4)
- net Rele4: now also IC?.16 (PTA7)
- net Bomba1: now reaches U?.5 (I5)
- net Bomba1: now also IC?.26 (PTB7)
- net Bomba2: now reaches U?.6 (I6)
- net Bomba2: now also IC?.25 (PTB6)
- net Aux1: now reaches U?.7 (I7)
- net Aux1: now also IC?.31 (PTC0)
- net Aux2: now reaches U?.8 (I8)
- net Aux2: now also IC?.32 (PTC1)
- net at Q?.1 (G): now also U?.7 (OUT_A)
- net at Q?.2 (D): now also J?.1 (Pin_1)
- net at J?.3 (Pin_3): now also R?.1 (x2)
- net Dht11: now reaches J?.1 (Pin_1)
- net TDS: now reaches C?.1, R?.2
- net TDS: now also IC?.18 (PTB1)
- net at Q?.1 (G): now also U?.5 (OUT_B)
- net at Q?.2 (D): now also J?.2 (Pin_2)
- new net: J?.1 (Pin_1), K?.12 (x4)
- new net: J?.2 (Pin_2), K?.14 (x4)
- new net: J?.3 (Pin_3), K?.11 (x4)
- new net DHT11: IC?.19 (PTB2)
- new net LDR: IC?.20 (PTB3)
- new net LUZ_A: IC?.23 (PTB4)
- new net LUZ_B: IC?.24 (PTB5)
- new net Luz_A: U?.2 (IN_A)
- new net Luz_B: U?.4 (IN_B)
- new net PH: C?.1, IC?.17 (PTB0), R?.2
- new net RX: IC?.9 (PTA1), J?.1 (Pin_1)
- new net SCL: IC?.11 (PTA3), J?.4 (Pin_4)
- new net SDA: IC?.10 (PTA2), J?.3 (Pin_3)
- new net TX: IC?.8 (PTA0), J?.2 (Pin_2)
Other:
- note removed: "-2.4k"
- note removed: "out"
- moved on the sheet: C?, J?, L?, Q?, R?, U?

Commit message: 1-7-2022
Parts:
- removed J?: Conn_01x04_Male, symbol Connector:Conn_01x04_Male
- removed J?: Conn_01x03, symbol Connector_Generic:Conn_01x03
- removed J?: Conn_01x08, symbol Connector_Generic:Conn_01x08
- removed SW?: SW_DIP_x03, symbol Switch:SW_DIP_x03
- added C7: 100nF, Capacitor_SMD:C_0603_1608Metric, symbol Device:C
- added J1: Bomba1, TerminalBlock:TerminalBlock_bornier-2_P5.08mm, symbol Connector_Generic:Conn_01x02
- added J11: Bomba2, TerminalBlock:TerminalBlock_bornier-2_P5.08mm, symbol Connector_Generic:Conn_01x02
- added J12: Aux1, TerminalBlock:TerminalBlock_bornier-2_P5.08mm, symbol Connector_Generic:Conn_01x02
- added J13: LCD, Connector_PinHeader_1.00mm:PinHeader_1x04_P1.00mm_Vertical, symbol Connector:Conn_01x04_Male
- added J14: Aux2, TerminalBlock:TerminalBlock_bornier-2_P5.08mm, symbol Connector_Generic:Conn_01x02
- added J15: Expansion, Connector_PinHeader_1.00mm:PinHeader_1x10_P1.00mm_Vertical, symbol Connector:Conn_01x10_Male
- added J16: NIVEL BAJO, TerminalBlock:TerminalBlock_bornier-2_P5.08mm, symbol Connector_Generic:Conn_01x02
- added J17: NIVEL ALTO, TerminalBlock:TerminalBlock_bornier-2_P5.08mm, symbol Connector_Generic:Conn_01x02
- added J18: LDR, TerminalBlock:TerminalBlock_bornier-2_P5.08mm, symbol Connector_Generic:Conn_01x02
- added J7: Rele4, TerminalBlock:TerminalBlock_bornier-3_P5.08mm, symbol Connector_Generic:Conn_01x03
- added R3, R4: 5k, Resistor_SMD:R_0603_1608Metric, symbol Device:R
- added R5, R6, R7: 1k, Resistor_SMD:R_0603_1608Metric, symbol Device:R
- added RV1: R_Potentiometer, Potentiometer_SMD:Potentiometer_Bourns_3314G_Vertical, symbol Device:R_Potentiometer
- added U4, U5: PC817, Package_DIP:DIP-4_W7.62mm, symbol Isolator:PC817
- added U6, U7: LM358, Package_SO:SOIC-8_3.9x4.9mm_P1.27mm, symbol Amplifier_Operational:LM358
- C1, C2, C3, C4, C5, C6: renamed from C?; footprint (none) -> Capacitor_SMD:C_0603_1608Metric
- J10: renamed from J?; value Conn_01x03 -> DHT11; footprint (none) -> TerminalBlock:TerminalBlock_bornier-3_P5.08mm
- J2: renamed from J?; value Conn_01x03 -> Rele1; footprint (none) -> TerminalBlock:TerminalBlock_bornier-3_P5.08mm
- J3: renamed from J?; value Conn_01x03 -> Luces; footprint (none) -> TerminalBlock:TerminalBlock_bornier-3_P5.08mm
- J4: renamed from J?; value Conn_01x03 -> Rele2; footprint (none) -> TerminalBlock:TerminalBlock_bornier-3_P5.08mm
- J5: renamed from J?; value Conn_01x03 -> TDS; footprint (none) -> TerminalBlock:TerminalBlock_bornier-3_P5.08mm
- J6: renamed from J?; value Conn_01x03 -> Rele3; footprint (none) -> TerminalBlock:TerminalBlock_bornier-3_P5.08mm
- J8: renamed from J?; value Conn_01x02 -> ENTRADA; footprint (none) -> TerminalBlock:TerminalBlock_bornier-2_P5.08mm
- J9: renamed from J?; value Conn_01x03 -> PH; footprint (none) -> TerminalBlock:TerminalBlock_bornier-3_P5.08mm
- L1: renamed from L?; footprint (none) -> Inductor_SMD:L_0603_1608Metric
- R1, R2: renamed from R?; footprint (none) -> Resistor_SMD:R_0603_1608Metric
- U1: renamed from U?; footprint (none) -> Package_SO:SOIC-18W_7.5x11.6mm_P1.27mm
- U2: renamed from U?; footprint (none) -> Package_SO:SOIC-8_3.9x4.9mm_P1.27mm
- gave numbers to parts that had none: 8
Connections:
- net +12V: now also U1.10 (COM), J1.2 (Pin_2), J11.2 (Pin_2), J12.2 (Pin_2), J14.2 (Pin_2)
- net +5V: now also J13.1 (Pin_1), J15.5 (Pin_5), J16.2 (Pin_2), J17.2 (Pin_2), J18.2 (Pin_2), R3.1, R4.1, U6.8 (V+), U7.8 (V+); no longer K1.A1, K2.A1, K3.A1, K4.A1, U1.10 (COM)
- net Aux1: now also IC1.24 (PTB5); no longer IC1.31 (PTC0)
- net Aux2: now also IC1.23 (PTB4); no longer IC1.32 (PTC1)
- net DHT11: now also IC1.4 (PTC5); no longer IC1.19 (PTB2)
- net GND: now also K1.A1, K2.A1, K3.A1, K4.A1, C7.2, J13.2 (Pin_2), J15.6 (Pin_6), J15.7 (Pin_7), RV1.2, RV1.3, U4.2, U4.3, U5.2, U5.3, U6.4 (V-), U7.4 (V-)
- net LUZ_A: now also IC1.32 (PTC1); no longer IC1.23 (PTB4)
- net LUZ_B: now also IC1.31 (PTC0); no longer IC1.24 (PTB5)
- net RX: now also J15.1 (Pin_1)
- net SCL: now also J13.4 (Pin_4), J15.4 (Pin_4)
- net SDA: now also J13.3 (Pin_3), J15.3 (Pin_3)
- net TX: now also J15.2 (Pin_2)
- net Nivel_bajo: now reaches IC1.1 (PTC2)
- net Nivel_bajo: now also R3.2, U4.4
- net Nivel_alto: now reaches IC1.2 (PTC3)
- net Nivel_alto: now also R4.2, U5.4
- net Digital: now reaches IC1.3 (PTC4)
- net Digital: now also J15.9 (Pin_9)
- net Digital_1: now reaches IC1.5 (PTC6)
- net Digital_1: now also J15.10 (Pin_10)
- net at U1.11 (O8): now also J14.1 (Pin_1)
- net at U1.12 (O7): now also J12.1 (Pin_1)
- net at U1.13 (O6): now also J11.1 (Pin_1)
- net at U1.14 (O5): now also J1.1 (Pin_1)
- net at J9.3 (Pin_3): now also U7.5 (+); no longer R2.1
- net at K4.11: now also J7.3 (Pin_3)
- net at K4.12: now also J7.1 (Pin_1)
- net at K4.14: now also J7.2 (Pin_2)
- net at R1.1: now also U6.1, U6.2 (-); no longer J5.3 (Pin_3)
- net LDR renamed ADC
- net ADC: now also J15.8 (Pin_8)
- new net: R2.1, U7.6 (-), U7.7
- new net: R7.1, U7.1, U7.2 (-)
- new net: J17.1 (Pin_1), R6.2
- new net: R5.1, U4.1
- new net: J16.1 (Pin_1), R5.2
- new net: J5.3 (Pin_3), U6.3 (+)
- new net: J18.1 (Pin_1), RV1.1, U7.3 (+)
- new net: R6.1, U5.1
- new net ldr: C7.1, IC1.19 (PTB2), R7.2
- no-connect marks 0 -> 12
Other:
- moved on the sheet: C2, C6, J10, J9, R1, R2

Commit message: 7-8-2022 itLA
Connections:
- net at J7.1 (Pin_1): now also K4.14; no longer K4.12
- net at J7.2 (Pin_2): now also K4.11; no longer K4.14
- net at J7.3 (Pin_3): now also K4.12; no longer K4.11
- net at J4.1 (Pin_1): now also K2.14; no longer K2.12
- net at J4.2 (Pin_2): now also K2.11; no longer K2.14
- net at J4.3 (Pin_3): now also K2.12; no longer K2.11
- net at K3.11: now also J6.2 (Pin_2); no longer J6.3 (Pin_3)
- net at K3.12: now also J6.3 (Pin_3); no longer J6.1 (Pin_1)
- net at K3.14: now also J6.1 (Pin_1); no longer J6.2 (Pin_2)
- net at J2.1 (Pin_1): now also K1.14; no longer K1.12
- net at J2.2 (Pin_2): now also K1.11; no longer K1.14
- net at J2.3 (Pin_3): now also K1.12; no longer K1.11
Other:
- moved on the sheet: J2, J4, J6, J7

Commit message: 15-7-2022
Parts:
- removed J1: Bomba1, TerminalBlock:TerminalBlock_bornier-2_P5.08mm, symbol Connector_Generic:Conn_01x02
- removed J15: Expansion, Connector_PinHeader_1.00mm:PinHeader_1x10_P1.00mm_Vertical, symbol Connector:Conn_01x10_Male
- removed U1: ULN2803A, Package_SO:SOIC-18W_7.5x11.6mm_P1.27mm, symbol Transistor_Array:ULN2803A
- added C10, C11: 100n, Capacitor_SMD:C_0201_0603Metric, symbol Device:C
- added C8, C9: 30p, Capacitor_SMD:C_0201_0603Metric, symbol Device:C
- added J1: Conn_01x12_Male, Connector_PinHeader_2.54mm:PinHeader_1x12_P2.54mm_Vertical, symbol Connector:Conn_01x12_Male
- added J15: Aux2, TerminalBlock:TerminalBlock_bornier-2_P5.08mm, symbol Connector_Generic:Conn_01x02
- added L2: 27n, Inductor_SMD:L_0805_2012Metric, symbol Device:L
- added R10, R11, R9: 10K, Resistor_SMD:R_0201_0603Metric, symbol Device:R
- added R8: 1M, Resistor_SMD:R_0201_0603Metric, symbol Device:R
- added RV2: Varistor_6V, Capacitor_SMD:C_0805_2012Metric, symbol Device:Varistor
- added U1, U8: ULN2003A, Package_SO:SOIC-16_3.9x9.9mm_P1.27mm, symbol Transistor_Array:ULN2003A
- added Y1: Crystal 4 MHz, Crystal:Crystal_HC49-4H_Vertical, symbol Device:Crystal
- C1, C4, C5: footprint Capacitor_SMD:C_0603_1608Metric -> Capacitor_SMD:C_0805_2012Metric
- C3: footprint Capacitor_SMD:C_0603_1608Metric -> Capacitor_SMD:C_0201_0603Metric
- J11: value Bomba2 -> Bomba1
- J12: value Aux1 -> Bomba2
- J14: value Aux2 -> Aux1
- L1: value L -> 4.7u; footprint Inductor_SMD:L_0603_1608Metric -> Inductor_SMD:L_Bourns_SRN6045TA
Connections:
- net +12V: now also K1.A1, K2.A1, K3.A1, K4.A1, J15.2 (Pin_2), U1.9 (COM), U8.9 (COM)
- net +5V: now also IC1.7 (VDD), C10.2, J1.9 (Pin_9), L2.1, R10.2, R11.2, RV2.1
- net ADC: now also J1.6 (Pin_6)
- net Aux1: now also U8.5 (I5)
- net Aux2: now also U8.6 (I6)
- net Bomba1: now also U8.1 (I1), U8.2 (I2)
- net Bomba2: now also U8.3 (I3), U8.4 (I4)
- net Digital: now also J1.7 (Pin_7)
- net Digital_1: now also J1.8 (Pin_8)
- net GND: now also IC1.22 (VSSA/VREFL), IC1.29 (VSS), IC1.6 (VSS), C10.1, C11.1, C8.1, C9.1, J1.12 (Pin_12), J1.5 (Pin_5), RV2.2, U1.8 (GND), U8.8 (GND); no longer K1.A1, K2.A1, K3.A1, K4.A1
- net RX: now also J1.1 (Pin_1)
- net Rele1: now also U1.1 (I1)
- net Rele2: now also U1.2 (I2)
- net Rele3: now also U1.3 (I3)
- net Rele4: now also U1.4 (I4)
- net SCL: now also J1.4 (Pin_4)
- net SDA: now also J1.3 (Pin_3)
- net TX: now also J1.2 (Pin_2)
- net at J14.1 (Pin_1): now also U8.12 (O5)
- net BKGD_PIN: now reaches IC1.12 (PTF1/~{RESET})
- net BKGD_PIN: now also J1.11 (Pin_11), R10.1
- net at IC1.21 (VDDA/VREFH): now also C11.2, L2.2
- net at IC1.27 (PTE5/XTAL): now also R9.2
- net at IC1.28 (PTE6/EXTAL): now also C9.2, R8.1, Y1.1
- net Reset_pin: now reaches IC1.30 (PTF0/BKGD/MS)
- net Reset_pin: now also J1.10 (Pin_10), R11.1
- net at J12.1 (Pin_1): now also U8.13 (O4), U8.14 (O3)
- net at J11.1 (Pin_1): now also U8.15 (O2), U8.16 (O1)
- net at K4.A2: now also U1.13 (O4)
- net at K3.A2: now also U1.14 (O3)
- net at K2.A2: now also U1.15 (O2)
- net at K1.A2: now also U1.16 (O1)
- new net: C8.2, R8.2, R9.1, Y1.2
- new net: J15.1 (Pin_1), U8.11 (O6)
- no-connect marks 12 -> 11
Other:
- moved on the sheet: IC1, J2, J3, J4, J6, J7, Q1, Q2, U2

Commit message: 7-15-2022 ITLA
Parts:
- removed J1: Conn_01x12_Male, Connector_PinHeader_2.54mm:PinHeader_1x12_P2.54mm_Vertical, symbol Connector:Conn_01x12_Male
- removed R9: 10K, Resistor_SMD:R_0201_0603Metric, symbol Device:R
- added J1: Conn_01x09_Male, Connector_PinSocket_2.54mm:PinSocket_1x09_P2.54mm_Vertical, symbol Connector:Conn_01x09_Male
- added SW1: SW_DIP_x04, symbol Switch:SW_DIP_x04
- J13: footprint Connector_PinHeader_1.00mm:PinHeader_1x04_P1.00mm_Vertical -> Connector_PinHeader_2.54mm:PinHeader_1x04_P2.54mm_Vertical
Connections:
- net +5V: now also J1.6 (Pin_6)
- net ADC: now also SW1.8
- net BKGD_PIN: now also J1.8 (Pin_8)
- net Digital: now also SW1.7
- net Digital_1: now also SW1.6
- net GND: now also J1.5 (Pin_5), J1.9 (Pin_9)
- net RX: now also J1.1 (Pin_1)
- net Reset_pin: now also J1.7 (Pin_7)
- net SCL: now also J1.4 (Pin_4)
- net SDA: now also J1.3 (Pin_3)
- net TX: now also J1.2 (Pin_2)
- net at IC1.27 (PTE5/XTAL): now also C8.2, R8.2, Y1.2
- net SW: now reaches C3.1, L1.1, U3.5 (SW)
- no-connect marks 11 -> 12
Other:
- moved on the sheet: R10, R11

Commit message: 22-7-2022
Connections:
- net Dht11 is gone; now on net GND: J10.1 (Pin_1)
- net Luz_A is gone; now on net luz a: U2.2 (IN_A)
- net Luz_B is gone; now on net luz b: U2.4 (IN_B)
- net +5V: now also J1.1 (Pin_1); no longer J1.6 (Pin_6)
- net Digital: now also IC1.19 (PTB2); no longer IC1.3 (PTC4)
- net GND: now also J1.2 (Pin_2); no longer J1.5 (Pin_5), J10.3 (Pin_3)
- net Nivel_alto: now also IC1.17 (PTB0); no longer IC1.2 (PTC3)
- net Nivel_bajo: now also IC1.18 (PTB1); no longer IC1.1 (PTC2)
- net PH: now also IC1.2 (PTC3); no longer IC1.17 (PTB0)
- net RX: now also J1.5 (Pin_5); no longer J1.1 (Pin_1)
- net Rele1: now also IC1.16 (PTA7); no longer IC1.13 (PTA4)
- net Rele2: now also IC1.15 (PTA6); no longer IC1.14 (PTA5)
- net Rele3: now also IC1.14 (PTA5); no longer IC1.15 (PTA6)
- net Rele4: now also IC1.13 (PTA4); no longer IC1.16 (PTA7)
- net TDS: now also IC1.1 (PTC2); no longer IC1.18 (PTB1)
- net TX: now also J1.6 (Pin_6); no longer J1.2 (Pin_2)
- net ldr: now also IC1.3 (PTC4); no longer IC1.19 (PTB2)
- net at U1.13 (O4): now also K1.A2; no longer K4.A2
- net at U1.14 (O3): now also K4.A2; no longer K3.A2
- net at U1.15 (O2): now also K3.A2; no longer K2.A2
- net at U1.16 (O1): now also K2.A2; no longer K1.A2
- net DHT11 renamed DHt11
- net DHt11: now also J10.3 (Pin_3)
- net LUZ_A renamed luz a
- net LUZ_B renamed luz b

Commit message: gg
Parts:
- removed RV1: R_Potentiometer, Potentiometer_SMD:Potentiometer_Bourns_3314G_Vertical, symbol Device:R_Potentiometer
- added C12: 4.7µ, Capacitor_SMD:C_0805_2012Metric, symbol pspice:CAP
- added C13: 100n, Capacitor_SMD:C_0201_0603Metric, symbol pspice:CAP
- added C14, C15: 100n, Capacitor_SMD:C_0201_0603Metric, symbol Device:C
- added R12, R13, R18, R19, R9: 10K, Resistor_SMD:R_0201_0603Metric, symbol Device:R
- added R14, R15, R16, R17: 10, Resistor_SMD:R_0201_0603Metric, symbol Device:R
- added R20: 100K, Resistor_SMD:R_0201_0603Metric, symbol Device:R
- J1: footprint Connector_PinSocket_2.54mm:PinSocket_1x09_P2.54mm_Vertical -> Connector_PinHeader_2.54mm:PinHeader_1x09_P2.54mm_Vertical
- SW1: footprint (none) -> Button_Switch_SMD:SW_DIP_SPSTx04_Slide_9.78x12.34mm_W8.61mm_P2.54mm
Connections:
- net +12V: now also U2.6 (V+), C12.1, C13.1
- net +5V: now also R12.1, R13.1, R9.1; no longer U2.6 (V+)
- net ADC: now also R9.2
- net Digital: now also R12.2
- net Digital_1: now also R13.2
- net GND: now also SW1.1, SW1.2, SW1.3, SW1.4, C12.2, C13.2, C14.2, C15.2, R18.2, R19.2, R20.2
- net Nivel_alto: now also C15.1
- net Nivel_bajo: now also C14.1
- net at U2.5 (OUT_B): now also R14.1, R15.1; no longer Q2.1 (G)
- net at U2.7 (OUT_A): now also R16.1, R17.1; no longer Q1.1 (G)
- net at J18.1 (Pin_1), U7.3 (+): now also R20.1
- new net: Q1.1 (G), R16.2, R17.2, R19.1
- new net: Q2.1 (G), R14.2, R15.2, R18.1
Other:
- moved on the sheet: J3, J5, J9, Q1, Q2
